File: MCP4725_v14.sch (EAGLE design)
At the start: 14 parts

Commit message: Addressed issues from first review
added new jumper packages
moved and rerouted to avoid cutting of silk text
added extra GND pad for VOUT
Parts:
- removed JP1: (no value), SparkFun:M05PTH
- removed SJ2: (no value), SparkFun-Passives:SOLDERJUMPER_2WAYPASTE2&3
- added GND: LOGO-SFESK, SparkFun:LOGO-SFESK
- added JP5: (no value), SparkFun-Connectors:M04PTH
- added JP6: M02PTH, SparkFun-Connectors:M02PTH
- SJ1: device SparkFun-Passives:SOLDERJUMPER_2WAYPASTE1&2&3 -> SparkFun-Passives:JUMPER-PAD-3-NC_BY_TRACE
- U$1: value LOGO-SFESK -> JUMPER-PAD-3-2OF3_NC_BY_PASTE; device SparkFun:LOGO-SFESK -> SparkFun-Passives:JUMPER-PAD-3-2OF3_NC_BY_PASTE
- renumbered U$2 to U1
Connections:
- net GND: now also JP5.4, JP6.1, U$1.3; no longer JP1.5, SJ2.3
- net N$3: now also U$1.2; no longer SJ2.2
- net SCL: now also JP5.1; no longer JP1.2
- net SDA: now also JP5.2; no longer JP1.3
- net VCC: now also JP5.3, U$1.1; no longer JP1.4, SJ2.1
- net VOUT: now also JP6.2; no longer JP1.1
Other:
- note added: "14"
- note removed: "V_14"
Changed lines of the file:
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@@
 <layer number="111" name="LPC17xx" color="7" fill="1" visible="yes" active="yes"/>
 <layer number="112" name="tSilk" color="7" fill="1" visible="yes" active="yes"/>
+<layer number="113" name="IDFDebug" color="4" fill="1" visible="yes" active="yes"/>
 <layer number="116" name="Patch_BOT" color="9" fill="4" visible="yes" active="yes"/>
 <layer number="121" name="_tsilk" color="7" fill="1" visible="yes" active="yes"/>
@@
 </classes>
 <parts>
-<part name="U$1" library="SparkFun" deviceset="LOGO-SFE" device="SK"/>
+<part name="GND" library="SparkFun" deviceset="LOGO-SFE" device="SK"/>
 <part name="C1" library="SparkFun" deviceset="CAP" device="0603-CAP" value="0.1uF"/>
 <part name="GND1" library="SparkFun" deviceset="GND" device=""/>
@@
 <part name="R2" library="SparkFun" deviceset="RESISTOR" device="0603-RES" value="10k"/>
 <part name="P+2" library="SparkFun" deviceset="VCC" device=""/>
-<part name="JP1" library="SparkFun" deviceset="M05" device="PTH"/>
 <part name="P+4" library="SparkFun" deviceset="VCC" device=""/>
 <part name="P+5" library="SparkFun" deviceset="VCC" device=""/>
 <part name="JP2" library="SparkFun" deviceset="FIDUCIAL" device="UFIDUCIAL"/>
 <part name="JP3" library="SparkFun" deviceset="FIDUCIAL" device="UFIDUCIAL"/>
-<part name="U$2" library="SparkFun-AnalogIC" deviceset="DAC_MCP4725" device="SOT-CP"/>
-<part name="SJ1" library="SparkFun-Passives" deviceset="SOLDERJUMPER_2WAY" device="PASTE1&amp;2&amp;3"/>
+<part name="U1" library="SparkFun-AnalogIC" deviceset="DAC_MCP4725" device="SOT-CP"/>
 <part name="GND2" library="SparkFun" deviceset="GND" device=""/>
 <part name="P+1" library="SparkFun" deviceset="VCC" device=""/>
-<part name="SJ2" library="SparkFun-Passives" deviceset="SOLDERJUMPER_2WAY" device="PASTE2&amp;3"/>
 <part name="STANDOFF1" library="SparkFun-Electromechanical" deviceset="STAND-OFF" device=""/>
 <part name="STANDOFF2" library="SparkFun-Electromechanical" deviceset="STAND-OFF" device=""/>
 <part name="FRAME2" library="SparkFun-Aesthetics" deviceset="FRAME-LETTER" device=""/>
 <part name="LOGO1" library="SparkFun-Aesthetics" deviceset="OSHW-LOGO" device="S"/>
+<part name="JP5" library="SparkFun-Connectors" deviceset="M04" device="PTH"/>
+<part name="JP6" library="SparkFun-Connectors" deviceset="M02" device="PTH"/>
+<part name="SJ1" library="SparkFun-Passives" deviceset="JUMPER-PAD-3-NC_BY_TRACE" device=""/>
+<part name="U$1" library="SparkFun-Passives" deviceset="JUMPER-PAD-3-2OF3_NC_BY_PASTE" device="" value=""/>
 </parts>
 <sheets>
@@
 VCC - 1100001</text>
 <text x="172.72" y="10.16" size="1.778" layer="91">Joel Bartlett</text>
-<text x="238.76" y="7.62" size="1.778" layer="91">V_14</text>
+<text x="238.76" y="7.62" size="1.778" layer="91">14</text>
 </plain>
 <instances>
-<instance part="U$1" gate="G$1" x="241.3" y="17.78"/>
+<instance part="GND" gate="G$1" x="241.3" y="17.78"/>
 <instance part="C1" gate="G$1" x="152.4" y="91.44"/>
 <instance part="GND1" gate="1" x="152.4" y="83.82"/>
@@
 <instance part="R2" gate="G$1" x="129.54" y="104.14" rot="R90"/>
 <instance part="P+2" gate="1" x="124.46" y="119.38"/>
-<instance part="JP1" gate="G$1" x="175.26" y="91.44"/>
 <instance part="P+4" gate="1" x="152.4" y="99.06"/>
 <instance part="P+5" gate="1" x="86.36" y="99.06"/>
 <instance part="JP2" gate="G$1" x="137.16" y="2.54"/>
 <instance part="JP3" gate="G$1" x="142.24" y="2.54"/>
-<instance part="U$2" gate="G$1" x="101.6" y="93.98"/>
-<instance part="SJ1" gate="G$1" x="124.46" y="111.76" rot="R270"/>
+<instance part="U1" gate="G$1" x="101.6" y="93.98"/>
 <instance part="GND2" gate="1" x="109.22" y="66.04"/>
 <instance part="P+1" gate="1" x="124.46" y="78.74"/>
-<instance part="SJ2" gate="G$1" x="116.84" y="73.66" rot="R270"/>
 <instance part="STANDOFF1" gate="G$1" x="137.16" y="12.7"/>
 <instance part="STANDOFF2" gate="G$1" x="142.24" y="12.7"/>
@@
 <instance part="FRAME2" gate="G$2" x="147.32" y="0"/>
 <instance part="LOGO1" gate="G$1" x="121.92" y="10.16"/>
+<instance part="JP5" gate="G$1" x="172.72" y="91.44"/>
+<instance part="JP6" gate="G$1" x="170.18" y="73.66"/>
+<instance part="SJ1" gate="G$1" x="124.46" y="111.76" rot="R270"/>
+<instance part="U$1" gate="G$1" x="116.84" y="73.66" rot="R270"/>
 </instances>
 <busses>
@@
 <wire x1="83.82" y1="93.98" x2="88.9" y2="93.98" width="0.1524" layer="91"/>
 <pinref part="GND5" gate="1" pin="GND"/>
-<pinref part="U$2" gate="G$1" pin="VSS"/>
+<pinref part="U1" gate="G$1" pin="VSS"/>
 </segment>
 <segment>
@@
 </segment>
 <segment>
-<wire x1="182.88" y1="96.52" x2="185.42" y2="96.52" width="0.1524" layer="91"/>
-<pinref part="JP1" gate="G$1" pin="5"/>
+<wire x1="177.8" y1="96.52" x2="185.42" y2="96.52" width="0.1524" layer="91"/>
 <label x="185.42" y="96.52" size="1.27" layer="95" xref="yes"/>
+<pinref part="JP5" gate="G$1" pin="4"/>
 </segment>
 <segment>
@@
 <wire x1="111.76" y1="73.66" x2="109.22" y2="73.66" width="0.1524" layer="91"/>
 <wire x1="109.22" y1="73.66" x2="109.22" y2="68.58" width="0.1524" layer="91"/>
-<pinref part="SJ2" gate="G$1" pin="3"/>
+<pinref part="U$1" gate="G$1" pin="3"/>
+</segment>
+<segment>
+<wire x1="177.8" y1="73.66" x2="180.34" y2="73.66" width="0.1524" layer="91"/>
+<label x="180.34" y="73.66" size="1.27" layer="95" xref="yes"/>
+<pinref part="JP6" gate="G$1" pin="1"/>
 </segment>
 </net>
@@
 <wire x1="86.36" y1="91.44" x2="86.36" y2="99.06" width="0.1524" layer="91"/>
 <pinref part="P+5" gate="1" pin="VCC"/>
-<pinref part="U$2" gate="G$1" pin="VDD"/>
+<pinref part="U1" gate="G$1" pin="VDD"/>
 </segment>
 <segment>
@@
 </segment>
 <segment>
-<pinref part="SJ1" gate="G$1" pin="2"/>
 <pinref part="P+2" gate="1" pin="VCC"/>
 <wire x1="124.46" y1="119.38" x2="124.46" y2="116.84" width="0.1524" layer="91"/>
+<pinref part="SJ1" gate="G$1" pin="2"/>
 </segment>
 <segment>
@@
 <wire x1="121.92" y1="73.66" x2="124.46" y2="73.66" width="0.1524" layer="91"/>
 <wire x1="124.46" y1="73.66" x2="124.46" y2="78.74" width="0.1524" layer="91"/>
-<pinref part="SJ2" gate="G$1" pin="1"/>
-</segment>
-<segment>
-<wire x1="182.88" y1="93.98" x2="185.42" y2="93.98" width="0.1524" layer="91"/>
-<pinref part="JP1" gate="G$1" pin="4"/>
+<pinref part="U$1" gate="G$1" pin="1"/>
+</segment>
+<segment>
+<wire x1="177.8" y1="93.98" x2="185.42" y2="93.98" width="0.1524" layer="91"/>
 <label x="185.42" y="93.98" size="1.27" layer="95" xref="yes"/>
+<pinref part="JP5" gate="G$1" pin="3"/>
 </segment>
 </net>
@@
 <pinref part="R1" gate="G$1" pin="1"/>
 <label x="132.08" y="93.98" size="1.27" layer="95" xref="yes"/>
-<pinref part="U$2" gate="G$1" pin="SCL"/>
-</segment>
-<segment>
-<wire x1="182.88" y1="88.9" x2="185.42" y2="88.9" width="0.1524" layer="91"/>
-<pinref part="JP1" gate="G$1" pin="2"/>
+<pinref part="U1" gate="G$1" pin="SCL"/>
+</segment>
+<segment>
+<wire x1="177.8" y1="88.9" x2="185.42" y2="88.9" width="0.1524" layer="91"/>
 <label x="185.42" y="88.9" size="1.27" layer="95" xref="yes"/>
+<pinref part="JP5" gate="G$1" pin="1"/>
 </segment>
 </net>
@@
 <pinref part="R2" gate="G$1" pin="1"/>
 <label x="132.08" y="91.44" size="1.27" layer="95" xref="yes"/>
-<pinref part="U$2" gate="G$1" pin="SDA"/>
-</segment>
-<segment>
-<wire x1="182.88" y1="91.44" x2="185.42" y2="91.44" width="0.1524" layer="91"/>
-<pinref part="JP1" gate="G$1" pin="3"/>
+<pinref part="U1" gate="G$1" pin="SDA"/>
+</segment>
+<segment>
+<wire x1="177.8" y1="91.44" x2="185.42" y2="91.44" width="0.1524" layer="91"/>
 <label x="185.42" y="91.44" size="1.27" layer="95" xref="yes"/>
+<pinref part="JP5" gate="G$1" pin="2"/>
 </segment>
 </net>
@@
 <segment>
 <pinref part="R2" gate="G$1" pin="2"/>
+<wire x1="129.54" y1="109.22" x2="129.54" y2="111.76" width="0.1524" layer="91"/>
 <pinref part="SJ1" gate="G$1" pin="1"/>
-<wire x1="129.54" y1="109.22" x2="129.54" y2="111.76" width="0.1524" layer="91"/>
 </segment>
 </net>
@@
 <segment>
 <pinref part="R1" gate="G$1" pin="2"/>
+<wire x1="119.38" y1="109.22" x2="119.38" y2="111.76" width="0.1524" layer="91"/>
 <pinref part="SJ1" gate="G$1" pin="3"/>
-<wire x1="119.38" y1="109.22" x2="119.38" y2="111.76" width="0.1524" layer="91"/>
 </segment>
 </net>
@@
 <wire x1="114.3" y1="96.52" x2="116.84" y2="96.52" width="0.1524" layer="91"/>
 <wire x1="116.84" y1="96.52" x2="116.84" y2="78.74" width="0.1524" layer="91"/>
-<pinref part="U$2" gate="G$1" pin="AO"/>
-<pinref part="SJ2" gate="G$1" pin="2"/>
+<pinref part="U1" gate="G$1" pin="AO"/>
+<pinref part="U$1" gate="G$1" pin="2"/>
 </segment>
 </net>
@@
 <wire x1="88.9" y1="96.52" x2="81.28" y2="96.52" width="0.1524" layer="91"/>
 <label x="81.28" y="96.52" size="1.27" layer="95" rot="R180" xref="yes"/>
-<pinref part="U$2" gate="G$1" pin="VOUT"/>
-</segment>
-<segment>
-<wire x1="182.88" y1="86.36" x2="185.42" y2="86.36" width="0.1524" layer="91"/>
-<pinref part="JP1" gate="G$1" pin="1"/>
-<label x="185.42" y="86.36" size="1.27" layer="95" xref="yes"/>
-</segment>
-</net>
+<pinref part="U1" gate="G$1" pin="VOUT"/>
+</segment>
+<segment>
+<wire x1="177.8" y1="76.2" x2="180.34" y2="76.2" width="0.1524" layer="91"/>
+<label x="180.34" y="76.2" size="1.27" layer="95" xref="yes"/>
+<pinref part="JP6" gate="G$1" pin="2"/>
+</segment>
+</net>
